Commit message: added move-base

File: src/robot_virat/urdf/my_robot.urdf (robot description, URDF)
Before this commit: robot my_robot, 6 links, 5 joints
Links:
- removed link body
- added link base_link, mass 5; collision mesh filename=package://robot_virat/meshes/body/bot2.dae; visual mesh filename=package://robot_virat/meshes/body/bot2.dae
Joints:
- joint camera_joint: parent body -> base_link
- joint castorer: parent body -> base_link
- joint dummy_joint: axis (none) -> 0 1 0; child body -> base_link
- joint wheeler1: parent body -> base_link
- joint wheeler2: parent body -> base_link
